File: Olimpiadas KiCad/Olimpiadas/Olimpiadas.kicad_pcb (KiCad board)
At the start: 2 copper layers, 32 parts, among them IC1 4047, Q1 2N2222, Q2 BD239, Q3 2N3772, Q4 2N2222, Q5 BD239, Q6 2N3772, U1 9.1v, U2 FUSIBLE

Commit message: PCB1
Parts:
- removed 12V1: CONN_01X02, EESTN5:BORNERA2_AZUL
- removed Transformador1: Conn_01X03, EESTN5:BORNERA3_AZUL
- added BZ1: Buzzer, EESTN5:Buzzer_12mm, F.Cu at (36.5, 167.8)
- added C7: C, EESTN5:CAP_ELEC_5x11mm, F.Cu at (115.6, 89.1)
- added C8: C, EESTN5:CAP_ELEC_5x11mm, F.Cu at (16.1, 159.7)
- added C9: C, EESTN5:CAP_ELEC_5x11mm, F.Cu at (17.1, 170.6)
- added D5: 1N4841, EESTN5:SOD80C, B.Cu at (122.6, 88.1)
- added F1: FUSE, EESTN5:FUSIBLE, F.Cu at (112.0, 41.0)
- added J1: PIN_meter, MacroLib:PIN_M, B.Cu at (37.7, 118.7)
- added J10: Cable_PAD, EESTN5:Tornillo_M3_8mm, F.Cu at (90.0, 40.0)
- added J11: Cable_PAD, EESTN5:Tornillo_M3_8mm, F.Cu at (90.0, 130.0)
- added J12: Cable_PAD, EESTN5:Tornillo_M3_8mm, F.Cu at (180.0, 40.0)
- added J13: Cable_PAD, EESTN5:Tornillo_M3_8mm, F.Cu at (180.0, 130.0)
- added J2: PIN_meter, MacroLib:PIN_M, B.Cu at (47.8, 131.5)
- added J3: PIN_meter, MacroLib:PIN_M, B.Cu at (44.0, 132.5)
- added J4: PIN_meter, MacroLib:PIN_M, B.Cu at (39.9, 125.6)
- added J5: PIN_meter, MacroLib:PIN_M, B.Cu at (144.5, 49.0)
- added J6: TB_1X2, EESTN5:BORNERA2_AZUL, F.Cu at (91.0, 52.8)
- added J7: TB_1X3, EESTN5:BORNERA3_AZUL, F.Cu at (226.5, 54.2)
- added J8: CONN_01X09, MacroLib:PIN_STRIP_9, F.Cu at (174.0, 63.0)
- added J9: CONN_01X03, EESTN5:Pin_Header_3, F.Cu at (179.0, 85.2)
- added Q10: MMBT2222, EESTN5:SOT23, B.Cu at (23.1, 153.5)
- added Q11: AO3401A, EESTN5:SOT23, B.Cu at (34.4, 148.8)
- added Q7: MMBT2222, EESTN5:SOT23, B.Cu at (106.7, 159.2)
- added Q8: MMBT2222, EESTN5:SOT23, B.Cu at (165.0, 61.8)
- added Q9: MMBT2222, EESTN5:SOT23, B.Cu at (13.8, 151.6)
- added R11: 10k, EESTN5:R_0805, B.Cu at (103.1, 156.1)
- added R12: R, EESTN5:R_0805, B.Cu at (107.4, 155.6)
- added R13: R, EESTN5:R_0805, B.Cu at (165.0, 65.8)
- added R14: R, EESTN5:R_0805, B.Cu at (122.2, 92.0)
- added R15: R, EESTN5:R_0805, B.Cu at (165.0, 57.5)
- added R16: R, EESTN5:R_0805, B.Cu at (19.3, 146.6)
- added R17: R, EESTN5:R_0805, B.Cu at (14.6, 146.7)
- added R18: R, EESTN5:R_0805, B.Cu at (124.5, 92.0)
- added R19: R, EESTN5:R_0805, B.Cu at (133.0, 79.8)
- added R20: R, EESTN5:R_0805, B.Cu at (133.0, 77.5)
- added R21: R, EESTN5:R_0805, B.Cu at (17.7, 151.0)
- added R22: R, EESTN5:R_0805, B.Cu at (25.0, 150.7)
- added R23: R, EESTN5:R_0805, B.Cu at (34.4, 154.3)
- added R24: 10k, EESTN5:R_0805, B.Cu at (142.8, 83.1)
- added R25: 10k, EESTN5:R_0805, B.Cu at (142.8, 81.1)
- added R26: 1k, EESTN5:R_0805, B.Cu at (142.8, 85.3)
- added R27: R, EESTN5:R_0805, B.Cu at (30.0, 151.7)
- added SW1: SW_PUSH, EESTN5:Pulsador_TH_4, F.Cu at (6.20, 159.9)
- added U3: LM358, EESTN5:DIP-8, F.Cu at (129.2, 83.0)
- 50K1: footprint EESTN5:Potenciometro -> EESTN5:TRIMER_V
- C1: value 10nf -> 100n
- C2: value 47uf -> 10nf; footprint EESTN5:CAP_ELEC_5x11mm -> EESTN5:CAP_0.1
- C3: value 100uf -> 47uf
- C4: value 100n -> 100uf; footprint EESTN5:CAP_0.1 -> EESTN5:CAP_ELEC_5x11mm
- C5: value 470n -> 100n
- C6: value 100n -> 470n
- D2: value 5A -> 1N4004
- D3: value 1N4004 -> 5A
- IC1: value 4047 -> CD4071BE; footprint Package_DIP:DIP-14_W7.62mm -> MacroLib:DIP-14
- Q1, Q4: value 2N2222 -> MMBT2222; footprint EESTN5:to92 -> EESTN5:SOT23; moved to B.Cu
- Q3, Q6: footprint Package_TO_SOT_THT:TO-3 -> MacroLib:TREE_HOLES
- R1: value 220 -> 22K; footprint EESTN5:RES0.3 -> EESTN5:R_0805; moved to B.Cu
- R10: value 22K -> 6.8 1W
- R2: value 100 1/2W -> 1K; footprint EESTN5:RES0.3 -> EESTN5:R_0805; moved to B.Cu
- R4, R7: footprint EESTN5:RES0.3 -> EESTN5:R_0805; moved to B.Cu
- R5: value 1K -> 6.8 1W
- R6: value 1K -> R; footprint EESTN5:RES0.3 -> EESTN5:R_0805; moved to B.Cu
- R8: value 6.8 1W -> 100 1/2W
- R9: value 6.8 1W -> 1K; footprint EESTN5:RES0.3 -> EESTN5:R_0805; moved to B.Cu
- U2: value FUSIBLE -> CD4047; footprint EESTN5:FUSIBLE -> MacroLib:DIP-14
- moved D1 111.7 mm to (164.5, 128.2)
- moved D3 96.1 mm to (101.2, 52.5)
- moved C2 93.2 mm to (133.5, 48.0), turned to 90 degrees
- moved D4 93.0 mm to (166.3, 159.3), turned to 90 degrees
- moved U2 91.6 mm to (129.0, 57.6), turned to 0 degrees
- moved Q4 90.2 mm to (151.9, 171.9), turned to 180 degrees
- moved R2 86.3 mm to (162.8, 99.5), turned to 180 degrees
- moved Q3 83.7 mm to (164.8, 122.5), turned to -90 degrees
- moved Q1 81.9 mm to (159.0, 107.5), turned to 180 degrees
- moved D2 80.0 mm to (105.0, 52.5), turned to -90 degrees
- moved R3 79.8 mm to (168.0, 105.0), turned to 0 degrees
- moved U1 79.8 mm to (122.7, 52.0), turned to -90 degrees
- moved C5 78.1 mm to (111.2, 56.2), turned to 90 degrees
- moved C1 73.6 mm to (121.2, 64.0), turned to 90 degrees
- moved R7 70.7 mm to (146.5, 166.0), turned to 180 degrees
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Connections:
- net Net-(D4-Pad2) renamed /T_B2
- C1 pad 2: GND -> Net-(C1-Pad2)
- C2 pad 1: Net-(C1-Pad1) -> +9V
- C3 pad 1: Net-(C3-Pad1) -> +9V
- C4 pad 1: Net-(C3-Pad1) -> /V_Diode
- C5 pad 1: Net-(C5-Pad1) -> /V_Diode
- C6 pad 1: Net-(C6-Pad1) -> /V_fuse
- C6 pad 2: Net-(C6-Pad2) -> GND
- D1 pad 1: Net-(C5-Pad1) -> GND
- D1 pad 2: Net-(C3-Pad1) -> /T_B1
- D2 pad 1: GND -> /V_fuse
- D2 pad 2: Net-(C5-Pad1) -> /V_Diode
- D3 pad 2: Net-(D3-Pad2) -> /V_fuse
- IC1 pad 1: Net-(C6-Pad2) -> /F_IC
- IC1 pad 10: Net-(IC1-Pad10) -> unconnected-(IC1-Pad10)
- IC1 pad 11: Net-(IC1-Pad11) -> unconnected-(IC1-Pad11)
- IC1 pad 12: GND -> unconnected-(IC1-Pad12)
- IC1 pad 14: Net-(C1-Pad1) -> VCC
- IC1 pad 2: Net-(50K1-Pad2) -> /F_TF
- IC1 pad 3: Net-(C6-Pad1) -> Net-(IC1-Pad3)
- IC1 pad 4: Net-(C1-Pad1) -> /F_general
- IC1 pad 5: Net-(C1-Pad1) -> Net-(IC1-Pad3)
- IC1 pad 6: Net-(C1-Pad1) -> /F_open
- IC1 pad 8: GND -> unconnected-(IC1-Pad8)
- IC1 pad 9: GND -> unconnected-(IC1-Pad9)
- Q2 pad 1: Net-(D3-Pad2) -> /T_B1
- Q2 pad 2: Net-(Q1-Pad3) -> Net-(Q1-Pad2)
- Q3 pad 1: Net-(D3-Pad2) -> /T_B1
- Q5 pad 2: Net-(Q4-Pad3) -> Net-(Q4-Pad2)
- R1 pad 2: Net-(C3-Pad1) -> Net-(50K1-Pad1)
- R10 pad 1: Net-(C6-Pad1) -> Net-(Q5-Pad3)
- R10 pad 2: Net-(50K1-Pad1) -> GND
- R2 pad 1: Net-(C3-Pad1) -> /Q
- R3 pad 1: Net-(C3-Pad1) -> /V_Diode
- R3 pad 2: Net-(Q4-Pad1) -> Net-(Q1-Pad3)
- R4 pad 1: Net-(Q4-Pad3) -> Net-(Q1-Pad2)
- R5 pad 1: Net-(IC1-Pad11) -> Net-(Q2-Pad3)
- R5 pad 2: Net-(Q4-Pad2) -> GND
- R6 pad 1: Net-(IC1-Pad10) -> +9V
- R6 pad 2: Net-(Q1-Pad2) -> /V_Diode
- R7 pad 1: Net-(Q1-Pad3) -> /N_Q
- R7 pad 2: GND -> Net-(Q4-Pad1)
- R8 pad 1: Net-(Q2-Pad3) -> /V_Diode
- R8 pad 2: GND -> Net-(Q4-Pad3)
- R9 pad 1: Net-(Q5-Pad3) -> Net-(Q4-Pad2)
- U1 pad 2: Net-(C1-Pad1) -> +9V
- U2 pad 1: Net-(C5-Pad1) -> Net-(C1-Pad2)
- U2 pad 2: VCC -> Net-(50K1-Pad2)
Routing:
- net GND: track 337.2 -> 0.00 mm
- net /T_B2: track 111.7 -> 0.00 mm
- net Net-(C1-Pad1): track 120.6 -> 11.5 mm
- net Net-(C5-Pad1): track 76.7 -> 0.00 mm
- net Net-(D3-Pad2): track 66.4 -> 0.00 mm
- net Net-(C6-Pad1): track 56.5 -> 0.00 mm
- net +9V: track 0.00 -> 54.3 mm
- net Net-(Q5-Pad3): track 52.6 -> 0.00 mm
- net /F_general: track 0.00 -> 47.9 mm
- net /OSC_OUT: track 0.00 -> 41.5 mm
- net VCC: track 11.8 -> 49.7 mm
- net Net-(Q2-Pad3): track 33.7 -> 0.00 mm
- net Net-(Q1-Pad3): track 33.7 -> 0.00 mm
- net /V_fuse: track 0.00 -> 32.1 mm
- net /V_Diode: track 0.00 -> 25.5 mm
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- added copper zone on B.Cu, net GND
Other:
- board outline added: 100 x 100 mm
