File: Olimpiadas KiCad/Olimpiadas/Olimpiadas.kicad_sch (KiCad schematic)
At the start: 32 parts, among them IC1 4047, Q1 2N2222, Q2 BD239, Q3 2N3772, Q4 2N2222, Q5 BD239, Q6 2N3772, U1 9.1v, U2 FUSIBLE

Commit message: PCB1
Parts:
- removed 12V1: CONN_01X02, EESTN5:BORNERA2_AZUL, symbol MacroLib:CONN_01X02
- removed IC1: 4047, Package_DIP:DIP-14_W7.62mm, symbol MacroLib2:4047
- removed Q1, Q4: 2N2222, EESTN5:to92, symbol EESTN5:BC338
- removed R1: 220, EESTN5:RES0.3, symbol EESTN5:R
- removed R3: 100 1/2W, EESTN5:RES0.3, symbol EESTN5:R
- removed R4, R5: 1K, EESTN5:RES0.3, symbol EESTN5:R
- removed Transformador1: Conn_01X03, EESTN5:BORNERA3_AZUL, symbol EESTN5:Conn_01X03
- removed U2: FUSIBLE, EESTN5:FUSIBLE, symbol EESTN5:FUSIBLE
- added BZ1: Buzzer, EESTN5:Buzzer_12mm, symbol EESTN5:Buzzer
- added C7, C8, C9: C, EESTN5:CAP_ELEC_5x11mm, symbol EESTN5:C
- added D5: 1N4841, EESTN5:SOD80C, symbol EESTN5:DIODE
- added F1: FUSE, EESTN5:FUSIBLE, symbol MacroLib:FUSE
- added IC1: CD4071BE, MacroLib:DIP-14, symbol MacroLib:CD4071BE
- added J1, J2, J3, J4, J5: PIN_meter, MacroLib:PIN_M, symbol MacroLib:PIN_meter
- added J10, J11, J12, J13: Cable_PAD, EESTN5:Tornillo_M3_8mm, symbol EESTN5:Cable_PAD
- added J6: TB_1X2, EESTN5:BORNERA2_AZUL, symbol EESTN5:TB_1X2
- added J7: TB_1X3, EESTN5:BORNERA3_AZUL, symbol EESTN5:TB_1X3
- added J8: CONN_01X09, MacroLib:PIN_STRIP_9, symbol MacroLib:CONN_01X09
- added J9: CONN_01X03, EESTN5:Pin_Header_3, symbol EESTN5:CONN_01X03
- added Q1, Q10, Q4, Q7, Q8, Q9: MMBT2222, EESTN5:SOT23, symbol MacroLib:MMBT2222
- added Q11: AO3401A, EESTN5:SOT23, symbol MacroLib:AO3401A
- added R10: 6.8 1W, EESTN5:RES0.3, symbol EESTN5:R
- added R11, R24, R25: 10k, EESTN5:R_0805, symbol EESTN5:R
- added R12, R13, R14, R15, R16, R17, R18, R19, R20, R21, R22, R23, R27, R6: R, EESTN5:R_0805, symbol EESTN5:R
- added R26: 1k, EESTN5:R_0805, symbol EESTN5:R
- added R7: 1K, EESTN5:R_0805, symbol EESTN5:R
- added R8: 100 1/2W, EESTN5:RES0.3, symbol EESTN5:R
- added SW1: SW_PUSH, EESTN5:Pulsador_TH_4, symbol EESTN5:SW_PUSH
- added U2: CD4047, MacroLib:DIP-14, symbol MacroLib:CD4047
- added U3: LM358, EESTN5:DIP-8, symbol MacroLib:LM358
- 50K1: footprint EESTN5:Potenciometro -> EESTN5:TRIMER_V
- Q3, Q6: footprint Package_TO_SOT_THT:TO-3 -> MacroLib:TREE_HOLES
- R1: renamed from R10; footprint EESTN5:RES0.3 -> EESTN5:R_0805
- R2: renamed from R6; footprint EESTN5:RES0.3 -> EESTN5:R_0805
- R4: renamed from R7; footprint EESTN5:RES0.3 -> EESTN5:R_0805
- R9: value 6.8 1W -> 1K; footprint EESTN5:RES0.3 -> EESTN5:R_0805
- renumbered C6 to C1, C1 to C2, C2 to C3, C3 to C4, C4 to C5, C5 to C6, D3 to D1, D1 to D2, D2 to D3, R2 to R3, R8 to R5
Connections:
- net GND: now also BZ1.2 (+), C9.2, IC1.7 (VSS), J6.2, J8.9, J9.3 (P3), Q10.2 (E), Q7.2 (E), Q8.2 (E), Q9.2 (E), R10.2, R14.2, R17.2, R18.2, R20.2, R21.2, R25.2, U2.12 (RETRIGGER), U2.7 (VSS), U2.8 (+TRIGGER), U2.9 (EXT.RESET), U3.4 (V-), U3.4 (V-)
- net VCC: now also F1.2, IC1.14 (VDD), J4.1, J6.1, J8.1, J8.7, J9.1 (P1), Q11.3, R12.1, R15.1, R19.1, R23.1, R24.1, R26.1, SW1.1, SW1.2, U3.8 (V+), U3.8 (V+)
- net V_fuse: now reaches C6.1, D2.1 (A), D3.2 (K)
- net V_fuse: now also F1.1, J3.1, J7.2, R11.1
- net +9V: now reaches C2.1, C3.1, U1.2 (K)
- net +9V: now also J8.8, R6.1, U2.14 (VDD), U2.4 (~{ASTABLE}), U2.5 (ASTABLE), U2.6 (-TRIGGER)
- net T_B1: now reaches D1.2 (K), Q2.1 (C), Q3.1 (C)
- net T_B1: now also J7.3
- net T_B2: now reaches D4.2 (K), Q5.1 (C), Q6.1 (C)
- net T_B2: now also J7.1
- net at Q5.2 (B): now also R9.1, Q4.2 (E)
- net at Q5.3 (E), Q6.2 (B): now also R10.1; no longer R9.1
- net at C1.1, R1.1: now also U2.3 (R-C_COMMON)
- net at 50K1.2, 50K1.3: now also U2.2 (R)
- net V_Diode: now reaches C4.1, C5.1, D2.2 (K), R3.1
- net V_Diode: now also R6.2, R8.1
- net at R3.2: now also Q1.3 (C)
- net Q: now reaches R2.1
- net Q: now also J1.1, U2.10 (Q)
- net at R2.2: now also Q1.1 (B)
- net at C1.2: now also U2.1 (C)
- net at Q2.2 (B), R4.1: now also Q1.2 (E)
- new net: R16.1, SW1.3, SW1.4
- new net: Q9.1 (B), R16.2, R17.1
- new net: C8.1, C9.1, Q10.1 (B), Q9.3 (C), R21.1, R22.2
- new net: Q10.3 (C), Q11.1, R23.2
- new net: Q4.3 (C), R8.2
- new net: BZ1.1 (-), R27.2
- new net: Q11.2, R22.1, R27.1
- new net: J9.2 (P2), R26.2, U3.6 (-)
- new net: R19.2, R20.1, U3.2 (-)
- new net: D5.2 (K), R18.1, U3.3 (+)
- new net: Q4.1 (B), R7.2
- new net: IC1.3 (J), IC1.5 (D)
- new net: C7.2, D5.1 (A), R14.1
- new net: R24.2, R25.1, U3.5 (+)
- new net: Q7.1 (B), R11.2
- new net: Q8.1 (B), R13.2
- new net F_IC: IC1.1 (B), J8.4, U3.1
- new net F_TF: IC1.2 (A), J8.5, U3.7
- new net F_general: C8.2, IC1.4 (K), J8.3, R13.1
- new net F_open: IC1.6 (C), J8.6, Q7.3 (C), R12.2
- new net N_Q: J2.1, R7.1, U2.11 (~{Q})
- new net OSC_OUT: C7.1, J5.1, U2.13 (OSC_OUT)
- new net R_normal: J8.2, Q8.3 (C), R15.2
Other:
- moved on the sheet: 50K1, C1, C2, C3, C4, C5, C6, D1, D2, D3, Q2, Q3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
